Commit message: Organized point cloud

File: rotors_description/urdf/rmf_obelix_base.xacro (robot description, xacro)
@@ -43,6 +43,6 @@
   <!-- Add an 0S0-128 lidar -->
   <xacro:include filename="$(find lidar_description)/urdf/OS0-128.urdf.xacro"/>
-  <xacro:OS0-128 parent="${namespace}/base_link" name="${namespace}/velodyne" topic="velodyne_points" hz="10" lasers="32" samples="440" collision_range="0.3" min_range="0.3" max_range="50.0">
-    <origin xyz="0 0 0.04" rpy="0 0 0" />
+  <xacro:OS0-128 parent="${namespace}/base_link" name="${namespace}/velodyne" topic="velodyne_points" hz="10" lasers="64" samples="512" collision_range="0.2" min_range="0.2" max_range="100.0" gpu="true" noise="0.01" organize_cloud="true">
+    <origin xyz="0.0 0 0.08" rpy="0 0 0" />
   </xacro:OS0-128>
 </robot>

Commit message: Added rpy in the spawn_mav and changed lidar specs

File: rotors_description/urdf/rmf_obelix_base.xacro (robot description, xacro)
@@ -43,6 +43,6 @@
   <!-- Add an 0S0-128 lidar -->
   <xacro:include filename="$(find lidar_description)/urdf/OS0-128.urdf.xacro"/>
-  <xacro:OS0-128 parent="${namespace}/base_link" name="${namespace}/velodyne" topic="velodyne_points" hz="10" lasers="64" samples="512" collision_range="0.2" min_range="0.2" max_range="100.0" gpu="true" noise="0.01" organize_cloud="true">
-    <origin xyz="0.0 0 0.08" rpy="0 0 0" />
+  <xacro:OS0-128 parent="${namespace}/base_link" name="${namespace}/ouster" topic="ouster_points" hz="10" lasers="64" samples="512" collision_range="0.3" min_range="0.3" max_range="50.0" gpu="true" organize_cloud="true">
+    <origin xyz="0.0 0 0.04" rpy="0 0 0" />
   </xacro:OS0-128>
 </robot>
